File: menestrel/kicad-project/menestel.kicad_pcb (KiCad board)
At the start: 2 copper layers, 94 x 59 mm, 31 parts, among them J1 Conn_01x01, J2 Conn_01x01, SW1 ПД11-5, U13 К155ЛА3, X1 СНП58-64, X2 СГ-3

Commit message: Правка мелких косяков Менестреля rev1
Other:
- outline, holes or cut-outs redrawn
- board text added: "Реплика {dblquote}Менестреля{dblquote} rev 2 Александр Алекссев, 2023 https://eax.me/menestrel/"
- board text removed: "Реплика {dblquote}Менестреля{dblquote} rev 1 Александр Алекссев, 2023 https://eax.me/menestrel/"
Changed lines of the file:
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@@
   (title_block
     (title "Реплика \"Менестреля\" ::: https://eax.me/menestrel/")
-    (date "2023-06-18")
-    (rev "1")
+    (date "2023-06-23")
+    (rev "2")
   )
   (layers
@@
   (gr_line (start 106.5 102) (end 100 102)
     (stroke (width 0.1) (type default)) (layer "Edge.Cuts"))
-  (gr_circle (center 189.75 96.75) (end 189.75 99)
+  (gr_circle (center 189.75 96.75) (end 192.25 96.75)
     (stroke (width 0.1) (type default)) (fill none) (layer "Edge.Cuts"))
   (gr_line (start 194 102) (end 187.5 102)
@@
   (gr_line (start 187.5 109) (end 106.5 109)
     (stroke (width 0.1) (type default)) (layer "Edge.Cuts"))
-  (gr_circle (center 104.25 96.75) (end 104.25 99)
+  (gr_circle (center 104.25 96.75) (end 106.75 96.75)
     (stroke (width 0.1) (type default)) (fill none) (layer "Edge.Cuts"))
   (gr_line (start 100 50) (end 194 50)
@@
   (gr_line (start 100 102) (end 100 50)
     (stroke (width 0.1) (type default)) (layer "Edge.Cuts"))
-  (gr_text "Реплика {dblquote}Менестреля{dblquote} rev 1\nАлександр Алекссев, 2023\nhttps://eax.me/menestrel/" (at 106.5 67 90) (layer "B.SilkS")
+  (gr_text "Реплика {dblquote}Менестреля{dblquote} rev 2\nАлександр Алекссев, 2023\nhttps://eax.me/menestrel/" (at 106.5 67 90) (layer "B.SilkS")
     (effects (font (size 1 1) (thickness 0.15)) (justify left bottom mirror))
   )
@@
   (segment (start 151 107.75) (end 154.25 107.75) (width 1.5) (layer "F.Cu") (net 3))
   (segment (start 136 100.25) (end 136 94) (width 1.5) (layer "F.Cu") (net 3))
-  (segment (start 186.25 95.45) (end 189.4 92.3) (width 1.5) (layer "F.Cu") (net 3))
+  (segment (start 186.25 95.45) (end 189.4 92.3) (width 1) (layer "F.Cu") (net 3))
   (segment (start 192.9 73.7) (end 192.9 65.9) (width 1.5) (layer "F.Cu") (net 3))
-  (segment (start 184.5 99.5) (end 186.25 97.75) (width 1.5) (layer "F.Cu") (net 3))
+  (segment (start 184.5 99.5) (end 186.25 97.75) (width 1) (layer "F.Cu") (net 3))
   (segment (start 133.25 107.25) (end 133.25 105.5) (width 1.5) (layer "F.Cu") (net 3))
   (segment (start 192.8 66) (end 185.2 66) (width 1.5) (layer "F.Cu") (net 3))
@@
   (segment (start 180.9 68.6) (end 180.64 68.6) (width 1.5) (layer "F.Cu") (net 3))
   (segment (start 150.75 103) (end 150.75 105.5) (width 1.5) (layer "F.Cu") (net 3))
-  (segment (start 189.4 92.3) (end 189.4 88.5) (width 1.5) (layer "F.Cu") (net 3))
+  (segment (start 189.4 92.3) (end 189.4 88.5) (width 1) (layer "F.Cu") (net 3))
   (segment (start 163.15 62.69) (end 163.15 53.85) (width 1.5) (layer "F.Cu") (net 3))
   (segment (start 133.75 107.75) (end 133.25 107.25) (width 1.5) (layer "F.Cu") (net 3))
   (segment (start 186.7 101.3) (end 187 101.6) (width 0.25) (layer "F.Cu") (net 3))
   (segment (start 184.8 83.9) (end 184.8 81.68) (width 1.5) (layer "F.Cu") (net 3))
-  (segment (start 186.25 97.75) (end 186.25 95.45) (width 1.5) (layer "F.Cu") (net 3))
+  (segment (start 186.25 97.75) (end 186.25 95.45) (width 1) (layer "F.Cu") (net 3))
   (segment (start 133.25 105.5) (end 133.25 103) (width 1.5) (layer "F.Cu") (net 3))
   (segment (start 141.5 99.5) (end 136.75 99.5) (width 1.5) (layer "F.Cu") (net 3))
